Commit message: Finished lesson 2.10

File: your_first_robot_with_ros/rosbots_description/urdf/rosbots.camera.gazebo.xacro (robot description, xacro)
@@ -31,4 +31,6 @@
      </plugin>
    </sensor>
+   <mu1>0.2</mu1>
+   <mu2>0.2</mu2>
  </gazebo>
 </robot>

File: your_first_robot_with_ros/rosbots_description/urdf/rosbots.gazebo.xacro (robot description, xacro)
@@ -21,3 +21,32 @@
     </plugin>
   </gazebo>
+  <gazebo reference="wheel_left_link">
+    <mu1>1.0</mu1>
+    <mu2>1.0</mu2>
+    <kp>1000000.0</kp>
+    <kd>100.0</kd>
+    <minDepth>0.001</minDepth>
+    <maxVel>1.0</maxVel>
+  </gazebo>
+  <gazebo reference="wheel_right_link">
+    <mu1>1.0</mu1>
+    <mu2>1.0</mu2>
+    <kp>1000000.0</kp>
+    <kd>100.0</kd>
+    <minDepth>0.001</minDepth>
+    <maxVel>1.0</maxVel>
+  </gazebo>
+  <gazebo reference="base_link">
+    <material>Gazebo/Blue</material>
+    <mu1>0.3</mu1>
+    <mu2>0.3</mu2>
+    <sensor type="contact" name="bumpers">
+      <always_on>1</always_on>
+      <update_rate>50.0</update_rate>
+      <visualize>true</visualize>
+      <contact>
+        <collision>base_footprint_collision_base_link</collision>
+      </contact>
+    </sensor>
+  </gazebo>
 </robot>
