Commit message: Finished lesson 2.6

File: your_first_robot_with_ros/rosbots_description/urdf/rosbots.xacro (robot description, xacro)
@@ -1,4 +1,5 @@
 <?xml version="1.0" encoding="utf-8"?>
 <robot name="rosbots" xmlns:xacro="http://www.ros.org/wiki/xacro">
+    <xacro:include filename="$(find rosbots_description)/urdf/rosbots.gazebo.xacro" />
     <link name="base_footprint"/>
     <!--The Base of the robot, forming the first level. -->
@@ -30,5 +31,5 @@
     </link>
     <!--The Base of the robot, forming the second level. -->
-<!--    <joint name="second_level_joint" type="fixed">
+    <joint name="second_level_joint" type="fixed">
       <origin xyz="0 0 0.68" rpy="0 0 0" />
       <parent link="base_link"/>
@@ -56,7 +57,6 @@
       </inertial>
     </link>
--->
     <!--The robot's micro-controller, on the second level. -->
-<!--     <joint name="mcu_joint" type="fixed">
+     <joint name="mcu_joint" type="fixed">
       <origin xyz="0.02 0.12 0.73" rpy="0 0 0" />
       <parent link="base_link"/>
@@ -84,7 +84,6 @@
       </inertial>
     </link>
--->
     <!--The robot's micro-controller, on the second level. -->
- <!--   <joint name="mcu_joint_1" type="fixed">
+   <joint name="mcu_joint_1" type="fixed">
       <origin xyz="0.02 0.12 0.83" rpy="0 0 0" />
       <parent link="base_link"/>
@@ -112,7 +111,6 @@
       </inertial>
     </link>
--->
     <!--The tandoff to support the micro-controllers on the second level. -->
- <!--   <joint name="stand_mcu1_joint" type="fixed">
+   <joint name="stand_mcu1_joint" type="fixed">
       <origin xyz="0.02 0.25 0.78" rpy="0 0 1.57" />
       <parent link="base_link"/>
@@ -133,7 +131,6 @@
       </collision>
     </link>
--->
     <!--The tandoff to support the micro-controllers on the second level. -->
- <!--   <joint name="stand_mcu2_joint" type="fixed">
+   <joint name="stand_mcu2_joint" type="fixed">
       <origin xyz="0.02 -0.1125 0.78" rpy="0 0 1.57" />
       <parent link="base_link"/>
@@ -154,7 +151,6 @@
       </collision>
     </link>
--->
    <!--The tandoff to support the micro-controllers on the second level. -->
- <!--  <joint name="stand_mcu3_joint" type="fixed">
+  <joint name="stand_mcu3_joint" type="fixed">
       <origin xyz="0.25 0.25 0.78" rpy="0 0 1.57" />
       <parent link="base_link"/>
@@ -175,7 +171,6 @@
       </collision>
     </link>
--->
     <!--The tandoff to support the micro-controllers on the second level. -->
- <!--   <joint name="stand_mcu4_joint" type="fixed">
+   <joint name="stand_mcu4_joint" type="fixed">
       <origin xyz="0.25 -0.1125 0.78" rpy="0 0 1.57" />
       <parent link="base_link"/>
@@ -196,7 +191,6 @@
       </collision>
     </link>
--->
     <!--Battery to supply power to the robot on the first level. -->
-<!--    <joint name="batery_joint" type="fixed">
+    <joint name="batery_joint" type="fixed">
       <origin xyz="1.2 0.2 0.43" rpy="0 0 1.57" />
       <parent link="base_link"/>
@@ -224,7 +218,6 @@
       </inertial>
     </link>
--->
     <!--Standoff to connect the first and second floors of the robot. -->
- <!--   <joint name="stand_1_joint" type="fixed">
+   <joint name="stand_1_joint" type="fixed">
       <origin xyz="0.5 0.4125 0.58" rpy="0 0 1.57" />
       <parent link="base_link"/>
@@ -252,7 +245,6 @@
       </inertial>
     </link>
--->
     <!--Standoff to connect the first and second floors of the robot. -->
- <!--   <joint name="stand_2_joint" type="fixed">
+   <joint name="stand_2_joint" type="fixed">
       <origin xyz="0.5 -0.2625 0.58" rpy="0 0 1.57" />
       <parent link="base_link"/>
@@ -280,7 +272,6 @@
       </inertial>
     </link>
-   -->
     <!--Standoff to connect the first and seconf floors of the robot. -->
- <!--   <joint name="stand_3_joint" type="fixed">
+   <joint name="stand_3_joint" type="fixed">
       <origin xyz="-0.4 0.4125 0.58" rpy="0 0 1.57" />
       <parent link="base_link"/>
@@ -301,7 +292,6 @@
       </collision>
     </link>
--->
     <!--Standoff to connect the first and seconf floors of the robot. -->
- <!--   <joint name="stand_4_joint" type="fixed">
+   <joint name="stand_4_joint" type="fixed">
       <origin xyz="-0.4 -0.2625 0.58" rpy="0 0 1.57" />
       <parent link="base_link"/>
@@ -322,6 +312,5 @@
       </collision>
     </link>
--->
-<!--Left Wheel of the robot. -->
+    <!--Left Wheel of the robot. -->
     <joint name="wheel_left_joint" type="continuous">
       <parent link="base_link"/>
@@ -354,6 +343,33 @@
     </link>
     <!--Right Wheel of the robot. -->
+    <joint name="wheel_right_joint" type="continuous">
+      <parent link="base_link"/>
+      <child link="wheel_right_link"/>
+      <origin xyz="0.15 -0.5625 0.30" rpy="-1.57 0 0"/>
+      <axis xyz="0 0 1"/>
+    </joint>
+    <link name="wheel_right_link">
+      <collision>
+        <geometry>
+         <cylinder length="0.20" radius="0.23"/>
+        </geometry>
+        <origin rpy="0.0 0.0 0" xyz="0 0 0.195"/>
+      </collision>
+      <visual name="visual">
+        <geometry>
+          <mesh filename="package://rosbots_description/meshes/wheel.dae" scale="8.0 8.0 8.0"/>
+        </geometry>
+        <origin rpy="0.0 0 0" xyz="0 0 0"/>
+      </visual>
+      <inertial>
+        <mass value="0.4" />
+        <origin xyz="0 0 0.3" />
+        <inertia ixx="0.001" ixy="0.0" ixz="0.0"
+                 iyy="0.001" iyz="0.0"
+                 izz="0.001" />
+      </inertial>
+    </link>
     <!--Caster Wheel of the robot. -->
-<!--    <joint name="caster_back_joint" type="fixed">
+    <joint name="caster_back_joint" type="fixed">
       <parent link="base_link"/>
       <child link="caster_back_link"/>
@@ -381,4 +397,3 @@
       </inertial>
     </link>
--->
 </robot>

Commit message: Completed Unit 2, removed inertials to stablize (stop the random rolling of) the robot in Gazebo.

File: your_first_robot_with_ros/rosbots_description/urdf/rosbots.xacro (robot description, xacro)
@@ -52,5 +52,5 @@
         <origin xyz="-0.52 -0.4 0.0" rpy="0 0 0"/>
       </collision>
-      <inertial>
+      <!--inertial>
         <origin xyz="0.01 0 0.7"/>
         <mass value="1.0"/>
@@ -58,5 +58,5 @@
                  iyy="0.01" iyz="0.0"
                  izz="0.03" />
-      </inertial>
+      </inertial-->
     </link>
     <!--The robot's micro-controller, on the second level. -->
@@ -79,5 +79,5 @@
         <origin xyz="0.9 -1.25 0" rpy="0 0 1.57"/>
       </collision>
-      <inertial>
+      <!--inertial>
         <origin xyz="0.01 0 0"/>
         <mass value="1.0"/>
@@ -85,5 +85,5 @@
                  iyy="0.019995" iyz="0.0"
                  izz="0.03675" />
-      </inertial>
+      </inertial-->
     </link>
     <!--The robot's micro-controller, on the second level. -->
@@ -106,5 +106,5 @@
         <origin xyz="0.9 -1.25 0" rpy="0 0 1.57"/>
       </collision>
-      <inertial>
+      <!--inertial>
         <origin xyz="0.01 0 0"/>
         <mass value="1.0"/>
@@ -112,5 +112,5 @@
                  iyy="0.019995" iyz="0.0"
                  izz="0.03675" />
-      </inertial>
+      </inertial-->
     </link>
     <!--The tandoff to support the micro-controllers on the second level. -->
@@ -213,5 +213,5 @@
         <origin xyz="0 4.5 0.05" rpy="1.57 0 1.57"/>
       </collision>
-      <inertial>
+      <!--inertial>
         <origin xyz="0.01 0 0"/>
         <mass value="1.0"/>
@@ -219,5 +219,5 @@
                  iyy="0.01" iyz="0.0"
                  izz="0.03" />
-      </inertial>
+      </inertial-->
     </link>
     <!--Standoff to connect the first and second floors of the robot. -->
@@ -240,11 +240,11 @@
         <origin rpy="0.0 0 0" xyz="0 0 0.0"/>
       </collision>
-      <inertial>
+      <!--inertial>
         <origin xyz="0.0 0 0"/>
         <mass value="1.0"/>
-        <inertia ixx="0.019995" ixy="0.0" ixz="0.0"
-                 iyy="0.019995" iyz="0.0"
-                 izz="0.03675" />
-      </inertial>
+       <inertia ixx="0.019995" ixy="0.0" ixz="0.0"
+                 iyy="0.019995" iyz="0.0"
+                 izz="0.03675" />
+      </inertial-->
     </link>
     <!--Standoff to connect the first and second floors of the robot. -->
@@ -267,5 +267,5 @@
         <origin rpy="0.0 0 0" xyz="0 0 0.0"/>
       </collision>
-      <inertial>
+      <!--inertial>
         <origin xyz="0.0 0 0"/>
         <mass value="1.0"/>
@@ -273,5 +273,5 @@
                  iyy="0.019995" iyz="0.0"
                  izz="0.03675" />
-      </inertial>
+      </inertial-->
     </link>
     <!--Standoff to connect the first and seconf floors of the robot. -->
@@ -294,4 +294,11 @@
         <origin rpy="0.0 0 0" xyz="0 0 0.0"/>
       </collision>
+      <!--inertial>
+        <origin xyz="0.0 0 0"/>
+        <mass value="1.0"/>
+       <inertia ixx="0.019995" ixy="0.0" ixz="0.0"
+                 iyy="0.019995" iyz="0.0"
+                 izz="0.03675" />
+      </inertial-->
     </link>
     <!--Standoff to connect the first and seconf floors of the robot. -->
@@ -314,4 +321,11 @@
         <origin rpy="0.0 0 0" xyz="0 0 0.0"/>
       </collision>
+      <!--inertial>
+        <origin xyz="0.0 0 0"/>
+        <mass value="1.0"/>
+       <inertia ixx="0.019995" ixy="0.0" ixz="0.0"
+                 iyy="0.019995" iyz="0.0"
+                 izz="0.03675" />
+      </inertial-->
     </link>
     <!--Left Wheel of the robot. -->
